File: ltc6820/ltc6820.kicad_sch (KiCad schematic)
At the start: 14 parts, among them J1 Conn_01x06_Pin, J2 Conn_01x02_Pin, T1 78613_3C

Commit message: Update: SPI Extender
Parts:
- removed JP1, JP2: SolderJumper_2_Bridged, Jumper:SolderJumper-2_P1.3mm_Open_RoundedPad1.0x1.5mm, symbol Jumper:SolderJumper_2_Bridged
- added R5: 10k, Resistor_THT:R_Axial_DIN0207_L6.3mm_D2.5mm_P10.16mm_Horizontal, symbol Device:R
- C1: value 27p -> 0.1u
- R4: value 1k -> 10k
Connections:
- net +3V3: now also C1.1, R5.1
- net MISO: now also R5.2
- net MOSI: now also R4.2
- net at T1.2: no longer C1.1
- no-connect marks 0 -> 1
Other:
- note removed: "not determined"
